Commit message: Acc

File: schunk_description/robots/schunk_arm_urdf.xacro (robot description, xacro)
@@ -8,5 +8,5 @@
   <xacro:include filename="$(find schunk_description)/urdf/sdh/sdh.urdf.xacro" />
    <!-- Create fixed base link (base of pedestal) -->
-  <link name="base_link" />
+  <link name="base_link"/>
   <link name="mid_link" />
   <joint name="base_mid_joint" type="fixed">

File: schunk_description/urdf/lwa4d/lwa4d.urdf.xacro (robot description, xacro)
@@ -58,5 +58,6 @@
     <!-- joint between arm_base_link and arm_1_link -->
     <joint name="${name}_1_joint" type="revolute">
-      <origin xyz="0 0 0" rpy="0 0 0" />
+      <!-- <origin xyz="0 0 0" rpy="0 0 0" /> -->
+      <origin xyz="0 0 0" rpy="0 0 -1.5708" />
       <parent link="${name}_base_link"/>
       <child link="${name}_1_link"/>
@@ -85,9 +86,11 @@
     <!-- joint between arm_1_link and arm_2_link -->
     <joint name="${name}_2_joint" type="revolute">
-      <origin xyz="0 0 0.240" rpy="-${M_PI/2} -${M_PI/2} 0"/>
+<!--      <origin xyz="0 0 0.240" rpy="-${M_PI/2} -${M_PI/2} 0"/> -->
+      <origin xyz="0 0 0.240" rpy="-${M_PI/2} -${M_PI} 0"/>
       <parent link="${name}_1_link"/>
       <child link="${name}_2_link"/>
       <xacro:axis_config invert="${invert_j2}"/>
-      <limit effort="216" velocity="0.43633" lower="${-2.14 + safety_offset}" upper="${2.14 - safety_offset}"/>
+      <limit effort="216" velocity="0.43633" lower="${-3.71 + safety_offset}" upper="${0.57 - safety_offset}"/>
+      <!-- <limit effort="216" velocity="0.43633" lower="${-2.14 + safety_offset}" upper="${2.14 - safety_offset}"/> -->
     </joint>
     <link name="${name}_2_link">
